File: hardware/pcb/mainboard/03-display.kicad_sch (KiCad schematic)
At the start: 21 parts, among them J4 FPC 24p 0.5mm - PANNEAU, J5 SECOURS DESPI-C579, Q4 Si1308EDL

Commit message: refactor(pcb): collapse to a single mainboard project
The two-perfboard design around the DevKitC-1 is gone; mainboard-v2 takes
the mainboard/ name and the -v2 suffix leaves every filename. The KiCad
project name is rewritten inside the instance blocks of all five sheets
too, otherwise KiCad drops the footprint assignments on open. ERC and DRC
still report 0 violations.

Add a Ground net class, split off Power, so GND carries its own via size
for the stitching and shows up in its own colour while routing. Its 0.2 mm
clearance is the neutral value: clearance resolves to the larger of the two
classes, so it never widens a gap on its own.

Drop the GPIO table from hardware/pcb/README.md rather than move it — the
netlist disagrees with it. PWR_HOLD no longer exists, PWR_SENSE is IO21 and
not IO41, and battery level comes from the BQ25896 over I2C instead of an
ADC. mainboard/README.md carries the pin plan that ships. wiring.md keeps
its bench-build pinout but stops attributing it to the deleted board.

hardware/bom.md, hardware/wiring.md and hardware/case/ still describe the
bench build, tracked as a TODO in the mainboard README.

Co-Authored-By: Claude Opus 5 <noreply@anthropic.com>
Other:
- title: Typoena mainboard v2 -> Typoena mainboard
Changed lines of the file:
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@@
 	(paper "A2")
 	(title_block
-		(title "Typoena mainboard v2")
+		(title "Typoena mainboard")
 		(date "2026-08-15")
 		(rev "A")
@@
 		)
 		(instances
-			(project "typoena-mainboard-v2"
+			(project "typoena-mainboard"
 				(path "/b1f0c5a2-7d34-4e19-9a6c-0f2e8d41c7b3/3a1c9e40-0003-4a00-9000-000000000003"
 					(reference "J4")
@@
 		)
 		(instances
-			(project "typoena-mainboard-v2"
+			(project "typoena-mainboard"
 				(path "/b1f0c5a2-7d34-4e19-9a6c-0f2e8d41c7b3/3a1c9e40-0003-4a00-9000-000000000003"
 					(reference "L4")
@@
 		)
 		(instances
-			(project "typoena-mainboard-v2"
+			(project "typoena-mainboard"
 				(path "/b1f0c5a2-7d34-4e19-9a6c-0f2e8d41c7b3/3a1c9e40-0003-4a00-9000-000000000003"
 					(reference "Q4")
@@
 		)
 		(instances
-			(project "typoena-mainboard-v2"
+			(project "typoena-mainboard"
 				(path "/b1f0c5a2-7d34-4e19-9a6c-0f2e8d41c7b3/3a1c9e40-0003-4a00-9000-000000000003"
 					(reference "R20")
@@
 		)
 		(instances
-			(project "typoena-mainboard-v2"
+			(project "typoena-mainboard"
 				(path "/b1f0c5a2-7d34-4e19-9a6c-0f2e8d41c7b3/3a1c9e40-0003-4a00-9000-000000000003"
 					(reference "R21")
@@
 		)
 		(instances
-			(project "typoena-mainboard-v2"
+			(project "typoena-mainboard"
 				(path "/b1f0c5a2-7d34-4e19-9a6c-0f2e8d41c7b3/3a1c9e40-0003-4a00-9000-000000000003"
 					(reference "D3")
@@
 		)
 		(instances
-			(project "typoena-mainboard-v2"
+			(project "typoena-mainboard"
 				(path "/b1f0c5a2-7d34-4e19-9a6c-0f2e8d41c7b3/3a1c9e40-0003-4a00-9000-000000000003"
 					(reference "D4")
@@
 		)
 		(instances
-			(project "typoena-mainboard-v2"
+			(project "typoena-mainboard"
 				(path "/b1f0c5a2-7d34-4e19-9a6c-0f2e8d41c7b3/3a1c9e40-0003-4a00-9000-000000000003"
 					(reference "D5")
@@
 		)
 		(instances
-			(project "typoena-mainboard-v2"
+			(project "typoena-mainboard"
 				(path "/b1f0c5a2-7d34-4e19-9a6c-0f2e8d41c7b3/3a1c9e40-0003-4a00-9000-000000000003"
 					(reference "C18")
@@
 		)
 		(instances
-			(project "typoena-mainboard-v2"
+			(project "typoena-mainboard"
 				(path "/b1f0c5a2-7d34-4e19-9a6c-0f2e8d41c7b3/3a1c9e40-0003-4a00-9000-000000000003"
 					(reference "C19")
@@
 		)
 		(instances
-			(project "typoena-mainboard-v2"
+			(project "typoena-mainboard"
 				(path "/b1f0c5a2-7d34-4e19-9a6c-0f2e8d41c7b3/3a1c9e40-0003-4a00-9000-000000000003"
 					(reference "C20")
@@
 		)
 		(instances
-			(project "typoena-mainboard-v2"
+			(project "typoena-mainboard"
 				(path "/b1f0c5a2-7d34-4e19-9a6c-0f2e8d41c7b3/3a1c9e40-0003-4a00-9000-000000000003"
 					(reference "C21")
@@
 		)
 		(instances
-			(project "typoena-mainboard-v2"
+			(project "typoena-mainboard"
 				(path "/b1f0c5a2-7d34-4e19-9a6c-0f2e8d41c7b3/3a1c9e40-0003-4a00-9000-000000000003"
 					(reference "C22")
@@
 		)
 		(instances
-			(project "typoena-mainboard-v2"
+			(project "typoena-mainboard"
 				(path "/b1f0c5a2-7d34-4e19-9a6c-0f2e8d41c7b3/3a1c9e40-0003-4a00-9000-000000000003"
 					(reference "C23")
@@
 		)
 		(instances
-			(project "typoena-mainboard-v2"
+			(project "typoena-mainboard"
 				(path "/b1f0c5a2-7d34-4e19-9a6c-0f2e8d41c7b3/3a1c9e40-0003-4a00-9000-000000000003"
 					(reference "C24")
@@
 		)
 		(instances
-			(project "typoena-mainboard-v2"
+			(project "typoena-mainboard"
 				(path "/b1f0c5a2-7d34-4e19-9a6c-0f2e8d41c7b3/3a1c9e40-0003-4a00-9000-000000000003"
 					(reference "C25")
@@
 		)
 		(instances
-			(project "typoena-mainboard-v2"
+			(project "typoena-mainboard"
 				(path "/b1f0c5a2-7d34-4e19-9a6c-0f2e8d41c7b3/3a1c9e40-0003-4a00-9000-000000000003"
 					(reference "C26")
@@
 		)
 		(instances
-			(project "typoena-mainboard-v2"
+			(project "typoena-mainboard"
 				(path "/b1f0c5a2-7d34-4e19-9a6c-0f2e8d41c7b3/3a1c9e40-0003-4a00-9000-000000000003"
 					(reference "C27")
@@
 		)
 		(instances
-			(project "typoena-mainboard-v2"
+			(project "typoena-mainboard"
 				(path "/b1f0c5a2-7d34-4e19-9a6c-0f2e8d41c7b3/3a1c9e40-0003-4a00-9000-000000000003"
 					(reference "R22")
@@
 		)
 		(instances
-			(project "typoena-mainboard-v2"
+			(project "typoena-mainboard"
 				(path "/b1f0c5a2-7d34-4e19-9a6c-0f2e8d41c7b3/3a1c9e40-0003-4a00-9000-000000000003"
 					(reference "R23")
@@
 		)
 		(instances
-			(project "typoena-mainboard-v2"
+			(project "typoena-mainboard"
 				(path "/b1f0c5a2-7d34-4e19-9a6c-0f2e8d41c7b3/3a1c9e40-0003-4a00-9000-000000000003"
 					(reference "J5")

Commit message: feat(pcb): route the mainboard and add the design checker
801 segments, 110 vias, five filled zones, no unconnected net. Board is
94x45 mm with four #6-32 corner holes; D2 dropped and GPIO 48 exposed on
J10; J4 mechanical pin tied to GND.

tools/check_pcb.py consolidates the checks that were improvised until now:
switching-node discipline, hot loops, decoupling, via-in-pad, fine-pitch
escapes, current capacity, schematic/PCB cross-checks.

Co-Authored-By: Claude Opus 5 <noreply@anthropic.com>
Parts:
- J4: symbol Connector_Generic:Conn_01x24 -> Connector_Generic_MountingPin:Conn_01x24_MountingPin
Connections:
- net GND: now also J4.MP (MountPin)
Other:
- moved on the sheet: C18, C19, C20, C21, C22, C23, C24, C25, C26, C27, D3, D4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
