File: hardware/pcb/mainboard/typoena-mainboard.kicad_pcb (KiCad board)
At the start: 4 copper layers, 94 x 45 mm, 95 parts, among them J1 BATTERIE JST-PH, J10 EXTENSION (non monte), J2 BOUTON contact JST-PH, J3 BOUTON LED JST-PH, J4 FPC 24p 0.5mm - PANNEAU, J5 SECOURS DESPI-C579, J6 USB-C CHARGE + PROG, J7 USB-C CLAVIER (hote), J8 microSD, J9 UART PROG, Q1 AO3401A, Q2 2N7002, Q3 2N7002, Q4 Si1308EDL, Q5 2N7002, Q6 2N7002, SW1 QON, SW2 RESET, SW3 BOOT, U1 ESP32-S3-WROOM-1-N16R8, U2 BQ25896RTW, U3 TPS63001DRCR, U4 TPS61023DRL, U5 CH343P

Commit message: PCB adjustments
Routing:
- net GND: track 82.1 -> 83.0 mm
- net USB_DM: track 88.4 -> 87.7 mm
Changed lines of the file:
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@@
 	)
 	(segment
+		(start 104.2 82.48125)
+		(end 105.0575 82.48125)
+		(width 0.6)
+		(layer "F.Cu")
+		(net "GND")
+	)
+	(segment
 		(start 87.2 67)
 		(end 86.9 66.7)
@@
 	)
 	(via
-		(at 105.0575 82.48125)
+		(at 104.2 82.48125)
 		(size 0.6)
 		(drill 0.3)
@@
 	)
 	(segment
-		(start 65.949314 59.835)
-		(end 59.24 59.835)
-		(width 0.2)
-		(layer "F.Cu")
-		(net "EPD_SCK")
-	)
-	(segment
-		(start 95.45 50.2)
-		(end 75.7 50.2)
-		(width 0.2)
-		(layer "F.Cu")
-		(net "EPD_SCK")
-	)
-	(segment
 		(start 131.25 50.634315)
 		(end 131.25 55.7)
@@
 	)
 	(segment
-		(start 75.675 50.225)
-		(end 75.559314 50.225)
-		(width 0.2)
-		(layer "F.Cu")
-		(net "EPD_SCK")
-	)
-	(segment
 		(start 103.25 56.12)
-		(end 101.37 56.12)
+		(end 101.275686 56.12)
 		(width 0.2)
 		(layer "F.Cu")
@@
 	)
 	(segment
-		(start 75.559314 50.225)
-		(end 65.949314 59.835)
+		(start 131.25 55.7)
+		(end 127.7 59.25)
 		(width 0.2)
 		(layer "F.Cu")
@@
 	)
 	(segment
-		(start 131.25 55.7)
-		(end 127.7 59.25)
+		(start 101.275686 56.12)
+		(end 95.930685 50.775)
 		(width 0.2)
 		(layer "F.Cu")
@@
 	)
 	(segment
-		(start 101.37 56.12)
-		(end 95.45 50.2)
+		(start 95.930685 50.775)
+		(end 75.211877 50.775)
+		(width 0.2)
+		(layer "F.Cu")
+		(net "EPD_SCK")
+	)
+	(segment
+		(start 75.211877 50.775)
+		(end 66.151877 59.835)
 		(width 0.2)
 		(layer "F.Cu")
@@
 	)
 	(segment
-		(start 75.7 50.2)
-		(end 75.675 50.225)
+		(start 66.151877 59.835)
+		(end 59.24 59.835)
 		(width 0.2)
 		(layer "F.Cu")
@@
 	)
 	(segment
-		(start 65.245 61.105)
-		(end 59.24 61.105)
+		(start 75.377563 51.175)
+		(end 65.447563 61.105)
 		(width 0.2)
 		(layer "F.Cu")
@@
 	)
 	(segment
-		(start 95.215 50.625)
-		(end 75.725 50.625)
+		(start 103.25 58.66)
+		(end 95.765 51.175)
 		(width 0.2)
 		(layer "F.Cu")
@@
 	)
 	(segment
-		(start 75.725 50.625)
-		(end 65.245 61.105)
+		(start 65.447563 61.105)
+		(end 59.24 61.105)
 		(width 0.2)
 		(layer "F.Cu")
@@
 	)
 	(segment
-		(start 103.25 58.66)
-		(end 95.215 50.625)
+		(start 130.85 50.8)
+		(end 130.85 55.5)
 		(width 0.2)
 		(layer "F.Cu")
@@
 	)
 	(segment
-		(start 130.85 50.8)
-		(end 130.85 55.5)
+		(start 95.765 51.175)
+		(end 75.377563 51.175)
 		(width 0.2)
 		(layer "F.Cu")
@@
 	)
 	(segment
-		(start 93.75 77.35)
-		(end 93.75 76.45)
-		(width 0.25)
-		(layer "F.Cu")
-		(net "USB_DP")
-	)
-	(segment
-		(start 91.786396 51.05)
-		(end 76.103604 51.05)
+		(start 75.553604 51.6)
+		(end 59.203604 67.95)
 		(width 0.25)
 		(layer "F.Cu")
@@
 	)
 	(segment
-		(start 100.05 81.686396)
-		(end 100.05 76.713604)
+		(start 93.75 77.35)
+		(end 93.75 76.45)
 		(width 0.25)
 		(layer "F.Cu")
@@
 	)
 	(segment
-		(start 59.203604 67.95)
-		(end 57.99 67.95)
+		(start 100.05 76.713604)
+		(end 95.85 72.513604)
 		(width 0.25)
 		(layer "F.Cu")
@@
 	)
 	(segment
-		(start 95.85 72.513604)
-		(end 95.85 55.113604)
+		(start 93.75 78.605)
+		(end 93.75 80.586396)
 		(width 0.25)
 		(layer "F.Cu")
@@
 	)
 	(segment
-		(start 99.786396 81.95)
-		(end 100.05 81.686396)
+		(start 95.113604 81.95)
+		(end 99.786396 81.95)
 		(width 0.25)
 		(layer "F.Cu")
@@
 	)
 	(segment
-		(start 95.85 55.113604)
-		(end 91.786396 51.05)
+		(start 95.85 72.513604)
+		(end 95.85 55.113604)
 		(width 0.25)
 		(layer "F.Cu")
@@
 	)
 	(segment
-		(start 76.103604 51.05)
-		(end 59.203604 67.95)
+		(start 100.05 81.686396)
+		(end 100.05 76.713604)
 		(width 0.25)
 		(layer "F.Cu")
@@
 	)
 	(segment
-		(start 95.113604 81.95)
-		(end 99.786396 81.95)
+		(start 94.8 78.555)
+		(end 94.8 77.79759)
+		(width 0.2)
+		(layer "F.Cu")
+		(net "USB_DP")
+	)
+	(segment
+		(start 99.786396 81.95)
+		(end 100.05 81.686396)
 		(width 0.25)
 		(layer "F.Cu")
@@
 	)
 	(segment
-		(start 94.8 78.555)
-		(end 94.8 77.79759)
+		(start 95 77.59759)
+		(end 95 76.7)
 		(width 0.2)
 		(layer "F.Cu")
@@
 	)
 	(segment
-		(start 100.05 76.713604)
-		(end 95.85 72.513604)
+		(start 92.336396 51.6)
+		(end 75.553604 51.6)
 		(width 0.25)
 		(layer "F.Cu")
@@
 	)
 	(segment
-		(start 95 77.59759)
-		(end 95 76.7)
+		(start 95 76.7)
+		(end 94.75 76.45)
 		(width 0.2)
 		(layer "F.Cu")
@@
 	)
 	(segment
-		(start 95 76.7)
-		(end 94.75 76.45)
-		(width 0.2)
+		(start 59.203604 67.95)
+		(end 57.99 67.95)
+		(width 0.25)
 		(layer "F.Cu")
 		(net "USB_DP")
 	)
 	(segment
-		(start 93.75 78.605)
-		(end 93.75 80.586396)
+		(start 95.85 55.113604)
+		(end 92.336396 51.6)
 		(width 0.25)
 		(layer "F.Cu")
@@
 	)
 	(segment
-		(start 76.29 51.5)
-		(end 58.765 69.025)
-		(width 0.25)
-		(layer "F.Cu")
-		(net "USB_DM")
-	)
-	(segment
 		(start 93.125 77.15)
 		(end 93.25 77.275)
@@
 	)
 	(segment
-		(start 97.3 74.6)
-		(end 95.4 72.7)
-		(width 0.25)
-		(layer "F.Cu")
-		(net "USB_DM")
-	)
-	(segment
-		(start 91.6 51.5)
-		(end 76.29 51.5)
-		(width 0.25)
-		(layer "F.Cu")
-		(net "USB_DM")
-	)
-	(segment
 		(start 95.3 81.5)
 		(end 99.6 81.5)
@@
 	)
 	(segment
-		(start 94.25 80.45)
-		(end 94.6 80.8)
+		(start 95.4 55.3)
+		(end 92.15 52.05)
 		(width 0.25)
 		(layer "F.Cu")
@@
 	)
 	(segment
-		(start 93.25 77.275)
-		(end 93.25 78.605)
+		(start 95.4 72.7)
+		(end 95.4 55.3)
 		(width 0.25)
 		(layer "F.Cu")
@@
 	)
 	(segment
-		(start 94.6 80.8)
-		(end 95.3 81.5)
+		(start 92.15 52.05)
+		(end 75.74 52.05)
 		(width 0.25)
 		(layer "F.Cu")
@@
 	)
 	(segment
-		(start 95.4 55.3)
-		(end 91.6 51.5)
+		(start 99.6 81.5)
+		(end 99.6 76.9)
 		(width 0.25)
 		(layer "F.Cu")
@@
 	)
 	(segment
-		(start 99.6 76.9)
-		(end 97.3 74.6)
+		(start 95.3 81.5)
+		(end 94.25 80.45)
 		(width 0.25)
 		(layer "F.Cu")
@@
 	)
 	(segment
-		(start 56.72 68.53)
-		(end 56.72 67.95)
+		(start 93.25 77.275)
+		(end 93.25 78.605)
 		(width 0.25)
 		(layer "F.Cu")
@@
 	)
 	(segment
-		(start 57.215 69.025)
-		(end 56.72 68.53)
+		(start 75.74 52.05)
+		(end 58.765 69.025)
 		(width 0.25)
 		(layer "F.Cu")
@@
 	)
 	(segment
-		(start 95.4 72.7)
-		(end 95.4 55.3)
+		(start 99.6 76.9)
+		(end 95.4 72.7)
 		(width 0.25)
 		(layer "F.Cu")
@@
 	)
 	(segment
-		(start 58.765 69.025)
-		(end 57.215 69.025)
+		(start 56.72 68.53)
+		(end 56.72 67.95)
 		(width 0.25)
 		(layer "F.Cu")
@@
 	)
 	(segment
-		(start 94.25 78.605)
-		(end 94.25 77.3)
+		(start 57.215 69.025)
+		(end 56.72 68.53)
 		(width 0.25)
 		(layer "F.Cu")
@@
 	)
 	(segment
-		(start 99.6 81.5)
-		(end 99.6 76.9)
+		(start 94.25 78.605)
+		(end 94.25 77.3)
 		(width 0.25)
 		(layer "F.Cu")
@@
 	)
 	(segment
-		(start 94.6 80.8)
-		(end 94.8 81)
+		(start 58.765 69.025)
+		(end 57.215 69.025)
 		(width 0.25)
 		(layer "F.Cu")
@@
 	)
 	(segment
-		(start 69.125 56.025)
-		(end 59.24 56.025)
+		(start 59.24 56.025)
+		(end 69.360837 56.025)
 		(width 0.25)
 		(layer "F.Cu")
@@
 	)
 	(segment
-		(start 75.583273 49.6)
-		(end 69.191637 55.991637)
+		(start 69.360837 56.025)
+		(end 75.785837 49.6)
 		(width 0.25)
 		(layer "F.Cu")
@@
 	)
 	(segment
-		(start 80.03 49.6)
-		(end 75.583273 49.6)
+		(start 75.785837 49.6)
+		(end 80.03 49.6)
 		(width 0.25)
 		(layer "F.Cu")
@@
 	)
 	(segment
-		(start 65.8 53.45)
-		(end 65.765 53.485)
-		(width 0.25)
-		(layer "F.Cu")
-		(net "IO48")
-	)
-	(segment
-		(start 70.21 53.45)
-		(end 65.8 53.45)
-		(width 0.25)
-		(layer "F.Cu")
-		(net "IO48")
-	)
-	(segment
-		(start 65.765 53.485)
+		(start 70.175 53.485)
 		(end 59.24 53.485)
 		(width 0.25)
@@
 	)
 	(via
-		(at 70.21 53.45)
+		(at 70.175 53.485)
 		(size 0.6)
 		(drill 0.3)
@@
 	)
 	(segment
-		(start 70.21 53.45)
+		(start 70.175 53.485)
 		(end 79.46 44.2)
 		(width 0.25)
