File: hardware/pcb/devboard/typoena-devboard.kicad_pcb (KiCad board)
At the start: 4 copper layers, 99 x 45 mm, 85 parts, among them J1 BATTERIE JST-PH, J11 DEVKITC-1 rangée gauche, J12 DEVKITC-1 rangée droite, J13 CLAVIER INTERNE, J2 BOUTON contact JST-PH, J3 BOUTON LED JST-PH, J4 FPC 24p 0.5mm - PANNEAU, J5 SECOURS DESPI-C579, J6 USB-C CHARGE + PROG, J7 USB-C CLAVIER (hote), J8 microSD, Q1 AO3401A, Q2 2N7002, Q3 2N7002, Q4 Si1308EDL, SW1 QON, U2 BQ25896RTW, U3 TPS63001DRCR, U4 TPS61023DRL

Commit message: Update mainboard
Connections:
- net USB_DM renamed USB_DN
Changed lines of the file:
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@@
 			(layers "F.Cu" "F.Mask" "F.Paste")
 			(roundrect_rratio 0.25)
-			(net "USB_DM")
+			(net "USB_DN")
 			(pinfunction "D-_A7")
 			(pintype "bidirectional")
@@
 			(layers "F.Cu" "F.Mask" "F.Paste")
 			(roundrect_rratio 0.25)
-			(net "USB_DM")
+			(net "USB_DN")
 			(pinfunction "D-_B7")
 			(pintype "bidirectional")
@@
 			(layers "*.Cu" "*.Mask")
 			(remove_unused_layers no)
-			(net "USB_DM")
+			(net "USB_DN")
 			(pinfunction "Pin_3_3")
 			(pintype "passive")
@@
 			(layers "*.Cu" "*.Mask")
 			(remove_unused_layers no)
-			(net "USB_DM")
+			(net "USB_DN")
 			(pinfunction "Pin_20_20")
 			(pintype "passive")
@@
 		(width 0.25)
 		(layer "F.Cu")
-		(net "USB_DM")
+		(net "USB_DN")
 	)
 	(segment
@@
 		(width 0.25)
 		(layer "F.Cu")
-		(net "USB_DM")
+		(net "USB_DN")
 	)
 	(segment
@@
 		(width 0.25)
 		(layer "F.Cu")
-		(net "USB_DM")
+		(net "USB_DN")
 	)
 	(segment
@@
 		(width 0.25)
 		(layer "F.Cu")
-		(net "USB_DM")
+		(net "USB_DN")
 	)
 	(segment
@@
 		(width 0.25)
 		(layer "F.Cu")
-		(net "USB_DM")
+		(net "USB_DN")
 	)
 	(via
@@
 		(drill 0.3)
 		(layers "F.Cu" "B.Cu")
-		(net "USB_DM")
+		(net "USB_DN")
 	)
 	(via
@@
 		(drill 0.3)
 		(layers "F.Cu" "B.Cu")
-		(net "USB_DM")
+		(net "USB_DN")
 	)
 	(segment
@@
 		(width 0.25)
 		(layer "B.Cu")
-		(net "USB_DM")
+		(net "USB_DN")
 	)
 	(segment
@@
 		(width 0.25)
 		(layer "B.Cu")
-		(net "USB_DM")
+		(net "USB_DN")
 	)
 	(segment
@@
 		(width 0.25)
 		(layer "B.Cu")
-		(net "USB_DM")
+		(net "USB_DN")
 	)
 	(segment
@@
 		(width 0.25)
 		(layer "B.Cu")
-		(net "USB_DM")
+		(net "USB_DN")
 	)
 	(segment
@@
 		(width 0.25)
 		(layer "B.Cu")
-		(net "USB_DM")
+		(net "USB_DN")
 	)
 	(segment
@@
 		(width 0.25)
 		(layer "B.Cu")
-		(net "USB_DM")
+		(net "USB_DN")
 	)
 	(segment
@@
 		(width 0.25)
 		(layer "B.Cu")
-		(net "USB_DM")
+		(net "USB_DN")
 	)
 	(segment
@@
 		(width 0.25)
 		(layer "B.Cu")
-		(net "USB_DM")
+		(net "USB_DN")
 	)
 	(segment
@@
 		(width 0.25)
 		(layer "B.Cu")
-		(net "USB_DM")
+		(net "USB_DN")
 	)
 	(segment
@@
 		(width 0.25)
 		(layer "B.Cu")
-		(net "USB_DM")
+		(net "USB_DN")
 	)
 	(segment
@@
 		(width 0.25)
 		(layer "B.Cu")
-		(net "USB_DM")
+		(net "USB_DN")
 	)
 	(segment
@@
 		(width 0.25)
 		(layer "B.Cu")
-		(net "USB_DM")
+		(net "USB_DN")
 	)
 	(segment
@@
 		(width 0.25)
 		(layer "B.Cu")
-		(net "USB_DM")
+		(net "USB_DN")
 	)
 	(segment
@@
 		(width 0.25)
 		(layer "B.Cu")
-		(net "USB_DM")
+		(net "USB_DN")
 	)
 	(segment
@@
 		(width 0.25)
 		(layer "B.Cu")
-		(net "USB_DM")
+		(net "USB_DN")
 	)
 	(segment
@@
 		(width 0.25)
 		(layer "B.Cu")
-		(net "USB_DM")
+		(net "USB_DN")
 	)
 	(segment
