File: hardware/pcb/mainboard/_restore_backup_2026-09-12T18-38-49-262/04-io.kicad_sch (KiCad schematic)
At the start: 30 parts, among them J13 CLAVIER INTERNE, J6 USB-C CHARGE + PROG, J7 USB-C CLAVIER (hote), J8 microSD, J9 UART PROG, Q5 2N7002, Q6 2N7002, U5 CH343P

Commit message: Update mainboard
Parts:
- removed TP1: GND, TestPoint:TestPoint_THTPad_D2.0mm_Drill1.0mm, symbol Connector:TestPoint
- removed TP10: IO39, TestPoint:TestPoint_THTPad_D1.5mm_Drill0.7mm, symbol Connector:TestPoint
- removed TP12: IO47, TestPoint:TestPoint_THTPad_D1.5mm_Drill0.7mm, symbol Connector:TestPoint
- removed TP13: IO48, TestPoint:TestPoint_THTPad_D1.5mm_Drill0.7mm, symbol Connector:TestPoint
- removed TP3: +3V3, TestPoint:TestPoint_THTPad_D2.0mm_Drill1.0mm, symbol Connector:TestPoint
- removed TP4: I2C_SDA, TestPoint:TestPoint_THTPad_D2.0mm_Drill1.0mm, symbol Connector:TestPoint
- removed TP5: I2C_SCL, TestPoint:TestPoint_THTPad_D2.0mm_Drill1.0mm, symbol Connector:TestPoint
- removed TP6: IO1, TestPoint:TestPoint_THTPad_D1.5mm_Drill0.7mm, symbol Connector:TestPoint
- removed TP7: IO2, TestPoint:TestPoint_THTPad_D1.5mm_Drill0.7mm, symbol Connector:TestPoint
- removed TP8: IO8, TestPoint:TestPoint_THTPad_D1.5mm_Drill0.7mm, symbol Connector:TestPoint
- removed TP9: IO9, TestPoint:TestPoint_THTPad_D1.5mm_Drill0.7mm, symbol Connector:TestPoint
- added J10: EXTENSION (non monte), Connector_PinHeader_2.54mm:PinHeader_1x12_P2.54mm_Vertical, symbol Connector_Generic:Conn_01x12
Connections:
- net +3V3: now also J10.2 (Pin_2)
- net GND: now also J10.1 (Pin_1)
- net I2C_SCL: now also J10.4 (Pin_4)
- net I2C_SDA: now also J10.3 (Pin_3)
- net IO1: now also J10.5 (Pin_5)
- net IO2: now also J10.6 (Pin_6)
- net IO39: now also J10.9 (Pin_9)
- net IO47: now also J10.11 (Pin_11)
- net IO48: now also J10.12 (Pin_12)
- net IO8: now also J10.7 (Pin_7)
- net IO9: now also J10.8 (Pin_8)
- net USB_DN renamed USB_DM
- net USB_PROG_DN renamed USB_PROG_DM
- new net IO42: J10.10 (Pin_10)
