File: hardware/pcb/mainboard/_restore_backup_2026-09-12T18-38-49-262/typoena-mainboard-v2.kicad_sch (KiCad schematic)
At the start: 0 parts

Commit message: Update mainboard
Other:
- note added: "FPC 24p, header DESPI de secours"
- note added: "microSD, pont USB-serie CH343P, extension"
- note removed: "FPC 24p"
- note removed: "USB-serie CH343P, extension"
- note removed: "clavier interne JST-PH, microSD, pont"
- title: Typoena mainboard -> Typoena mainboard v2
Changed lines of the file:
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@@
 	(paper "A4")
 	(title_block
-		(title "Typoena mainboard")
+		(title "Typoena mainboard v2")
 		(date "2026-08-15")
 		(rev "A")
@@
 		(comment 2 "Connectivite inter-feuilles par etiquettes globales")
 	)
-	(text "USB-serie CH343P, extension"
-		(exclude_from_sim no)
-		(at 130.81 166.02 0)
-		(effects
-			(font
-				(size 1.5 1.5)
-				(bold yes)
-			)
-			(justify left bottom)
-		)
-	)
 	(text "IO - USB-C charge/prog, USB-C clavier (hote),"
 		(exclude_from_sim no)
@@
 		)
 	)
+	(text "Alimentation - BQ25896 (charge + power path"
+		(exclude_from_sim no)
+		(at 30.48 93.98 0)
+		(effects
+			(font
+				(size 1.5 1.5)
+				(bold yes)
+			)
+			(justify left bottom)
+		)
+	)
+	(text "microSD, pont USB-serie CH343P, extension"
+		(exclude_from_sim no)
+		(at 130.81 163.02 0)
+		(effects
+			(font
+				(size 1.5 1.5)
+				(bold yes)
+			)
+			(justify left bottom)
+		)
+	)
+	(text "decouplage"
+		(exclude_from_sim no)
+		(at 130.81 96.98 0)
+		(effects
+			(font
+				(size 1.5 1.5)
+				(bold yes)
+			)
+			(justify left bottom)
+		)
+	)
+	(text "NVDC), TPS63001 3V3, TPS61023 5V clavier, rail"
+		(exclude_from_sim no)
+		(at 30.48 96.98 0)
+		(effects
+			(font
+				(size 1.5 1.5)
+				(bold yes)
+			)
+			(justify left bottom)
+		)
+	)
+	(text "FPC 24p, header DESPI de secours"
+		(exclude_from_sim no)
+		(at 30.48 163.02 0)
+		(effects
+			(font
+				(size 1.5 1.5)
+				(bold yes)
+			)
+			(justify left bottom)
+		)
+	)
+	(text "Ecran GDEY0579T93 - etage de puissance du §9,"
+		(exclude_from_sim no)
+		(at 30.48 160.02 0)
+		(effects
+			(font
+				(size 1.5 1.5)
+				(bold yes)
+			)
+			(justify left bottom)
+		)
+	)
+	(text "uSD commute, bouton"
+		(exclude_from_sim no)
+		(at 30.48 99.98 0)
+		(effects
+			(font
+				(size 1.5 1.5)
+				(bold yes)
+			)
+			(justify left bottom)
+		)
+	)
 	(text "MCU - ESP32-S3-WROOM-1-N16R8, strapping,"
 		(exclude_from_sim no)
 		(at 130.81 93.98 0)
-		(effects
-			(font
-				(size 1.5 1.5)
-				(bold yes)
-			)
-			(justify left bottom)
-		)
-	)
-	(text "decouplage"
-		(exclude_from_sim no)
-		(at 130.81 96.98 0)
-		(effects
-			(font
-				(size 1.5 1.5)
-				(bold yes)
-			)
-			(justify left bottom)
-		)
-	)
-	(text "Alimentation - BQ25896 (charge + power path"
-		(exclude_from_sim no)
-		(at 30.48 93.98 0)
-		(effects
-			(font
-				(size 1.5 1.5)
-				(bold yes)
-			)
-			(justify left bottom)
-		)
-	)
-	(text "uSD commute, bouton"
-		(exclude_from_sim no)
-		(at 30.48 99.98 0)
-		(effects
-			(font
-				(size 1.5 1.5)
-				(bold yes)
-			)
-			(justify left bottom)
-		)
-	)
-	(text "Ecran GDEY0579T93 - etage de puissance du §9,"
-		(exclude_from_sim no)
-		(at 30.48 160.02 0)
-		(effects
-			(font
-				(size 1.5 1.5)
-				(bold yes)
-			)
-			(justify left bottom)
-		)
-	)
-	(text "clavier interne JST-PH, microSD, pont"
-		(exclude_from_sim no)
-		(at 130.81 163.02 0)
-		(effects
-			(font
-				(size 1.5 1.5)
-				(bold yes)
-			)
-			(justify left bottom)
-		)
-	)
-	(text "FPC 24p"
-		(exclude_from_sim no)
-		(at 30.48 163.02 0)
-		(effects
-			(font
-				(size 1.5 1.5)
-				(bold yes)
-			)
-			(justify left bottom)
-		)
-	)
-	(text "NVDC), TPS63001 3V3, TPS61023 5V clavier, rail"
-		(exclude_from_sim no)
-		(at 30.48 96.98 0)
 		(effects
 			(font
@@
 		)
 		(instances
-			(project "typoena-mainboard"
+			(project "typoena-mainboard-v2"
 				(path "/b1f0c5a2-7d34-4e19-9a6c-0f2e8d41c7b3"
 					(page "2")
@@
 		)
 		(instances
-			(project "typoena-mainboard"
+			(project "typoena-mainboard-v2"
 				(path "/b1f0c5a2-7d34-4e19-9a6c-0f2e8d41c7b3"
 					(page "3")
@@
 		)
 		(instances
-			(project "typoena-mainboard"
+			(project "typoena-mainboard-v2"
 				(path "/b1f0c5a2-7d34-4e19-9a6c-0f2e8d41c7b3"
 					(page "4")
@@
 		)
 		(instances
-			(project "typoena-mainboard"
+			(project "typoena-mainboard-v2"
 				(path "/b1f0c5a2-7d34-4e19-9a6c-0f2e8d41c7b3"
 					(page "5")
