File: hardware/pcb/mainboard/_restore_backup_2026-09-12T19-00-22-220/typoena-mainboard.kicad_pcb (KiCad board)
At the start: 4 copper layers, 99 x 45 mm, 105 parts, among them J1 BATTERIE JST-PH, J13 CLAVIER INTERNE, J2 BOUTON contact JST-PH, J3 BOUTON LED JST-PH, J4 FPC 24p 0.5mm - PANNEAU, J6 USB-C CHARGE + PROG, J7 USB-C CLAVIER (hote), J8 microSD, J9 UART PROG, Q1 AO3401A, Q2 2N7002, Q3 2N7002, Q4 Si1308EDL, Q5 2N7002, Q6 2N7002, SW1 QON, SW2 RESET, SW3 BOOT, U1 ESP32-S3-WROOM-1-N16R8, U2 BQ25896RTW, U3 TPS63001DRCR, U4 TPS61023DRL, U5 CH343P

Commit message: Update mainboard
Parts:
- removed TP1: GND, TestPoint:TestPoint_THTPad_D2.0mm_Drill1.0mm
- removed TP10: IO39, TestPoint:TestPoint_THTPad_D1.5mm_Drill0.7mm
- removed TP12: IO47, TestPoint:TestPoint_THTPad_D1.5mm_Drill0.7mm
- removed TP13: IO48, TestPoint:TestPoint_THTPad_D1.5mm_Drill0.7mm
- removed TP3: +3V3, TestPoint:TestPoint_THTPad_D2.0mm_Drill1.0mm
- removed TP4: I2C_SDA, TestPoint:TestPoint_THTPad_D2.0mm_Drill1.0mm
- removed TP5: I2C_SCL, TestPoint:TestPoint_THTPad_D2.0mm_Drill1.0mm
- removed TP6: IO1, TestPoint:TestPoint_THTPad_D1.5mm_Drill0.7mm
- removed TP7: IO2, TestPoint:TestPoint_THTPad_D1.5mm_Drill0.7mm
- removed TP8: IO8, TestPoint:TestPoint_THTPad_D1.5mm_Drill0.7mm
- removed TP9: IO9, TestPoint:TestPoint_THTPad_D1.5mm_Drill0.7mm
- added J10: EXTENSION (non monte), Connector_PinHeader_2.54mm:PinHeader_1x12_P2.54mm_Vertical, F.Cu at (-80.0, 43.0)
- moved J9 135.0 mm to (-88.0, 37.7), turned to 180 degrees
- moved C29 0.37 mm to (34.7, 80.6)
Routing:
- net EN: track 51.7 -> 17.7 mm, vias 5 -> 2
- net UART_RX: track 71.0 -> 45.8 mm
- net UART_TX: track 65.4 -> 43.1 mm
- net IO8: track 13.6 -> 0.00 mm, vias 1 -> 0
- net IO1: track 10.9 -> 0.00 mm
- net IO2: track 8.64 -> 0.00 mm
- net VBUS: track 67.2 -> 59.2 mm, vias 2 -> 0
- net I2C_SDA: track 62.2 -> 56.1 mm, vias 4 -> 3
- net IO0: track 40.6 -> 36.3 mm
- net IO9: track 4.16 -> 0.00 mm
- net IO48: track 4.06 -> 0.00 mm
- net I2C_SCL: track 55.6 -> 51.6 mm, vias 4 -> 3
- net IO47: track 3.36 -> 0.00 mm
- net IO39: track 2.93 -> 0.00 mm
- net EPD_CS: track 125.1 -> 127.8 mm
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